File: kicad/yamashnik.sch (KiCad schematic (older format))
At the start: 13 parts, among them J1 USB_AM_PCB, P1 CONN_5, P2 CONN_4, U1 6N137, U2 6N138, U3 CP2102

Commit message: update schematic, added pdf drawing
Other:
- note added: "Cable/male DIN5 connector"
- moved on the sheet: C1, C2, C3, J1, P1, P2, R1, R2, R3, R4, U1, U2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
